File: REV11-KI-THT-SMD/REV11-KI-THT-SMD.kicad_pcb (KiCad board)
At the start: 2 copper layers, 114.3 x 73 mm, 40 parts, among them J1 EJ508A (PWR), J2 54-00298, P1 SPADE, P2 SPADE, Q1 2N3904, U1 NJM78M05FA, U2 LMC555CN, U3 LMC555CN, U4 STQ, U5 ESP32-C3-DEVKITC-02HOLES

Commit message: new files, readme, etc
Routing:
- net Net-(U3-DIS): track 11.8 -> 15.0 mm
Changed lines of the file:
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@@
 	)
 	(paper "A4")
+	(title_block
+		(title "REV-11")
+		(company "Designed by Rhett Applestone")
+		(comment 1 "Project of MIT-NSE")
+	)
 	(layers
 		(0 "F.Cu" signal)
@@
 			(drillshape 0)
 			(scaleselection 1)
-			(outputdirectory "/home/rhett/Desktop/REV-10-KI-THT-SMD-OUTPUTS/")
+			(outputdirectory "/home/rhett/Desktop/REV11-KI-THT-SMD-OUTPUTS")
 		)
 	)
@@
 	)
 	(segment
+		(start 135.44 85.535)
+		(end 133.58 83.675)
+		(width 0.8128)
+		(layer "F.Cu")
+		(net 6)
+	)
+	(segment
+		(start 136.01 85.535)
+		(end 135.44 85.535)
+		(width 0.8128)
+		(layer "F.Cu")
+		(net 6)
+	)
+	(segment
