File: REV11-KI-THT-SMD/REV11-KI-THT-SMD.kicad_sch (KiCad schematic)
At the start: 36 parts, among them J1 EJ508A (PWR), J2 54-00298, P1 SPADE, P2 SPADE, Q1 2N3904, U1 NJM78M05FA, U2 LMC555CN, U3 LMC555CN, U4 STQ, U5 ESP32-C3-DEVKITC-02HOLES

Commit message: new files, readme, etc
Changed lines of the file:
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@@
 	(text "HIGH VOLTAGE SUPPLY"
 		(exclude_from_sim no)
-		(at 173.99 51.308 0)
+		(at 171.958 51.308 0)
 		(effects
 			(font
